Commit message: Update kinect_v2.urdf.xacro

File: kinect_v2/urdf/kinect_v2.urdf.xacro (robot description, xacro)
@@ -19,5 +19,5 @@
                 <origin xyz="0 0 0" rpy="0 0 0" />
                 <geometry>
-                    <mesh filename="package://dhbot_description/meshes/kinect2.STL" />
+                    <mesh filename="package://kinect_v2/meshes/kinect2.STL" />
                 </geometry>
                 <material name="">
@@ -28,5 +28,5 @@
                 <origin xyz="0 0 0" rpy="0 0 0" />
                 <geometry>
-                    <mesh filename="package://dhbot_description/meshes/kinect2.STL" />
+                    <mesh filename="package://kinect_v2/meshes/kinect2.STL" />
                 </geometry>
             </collision>
